Commit message: Changed lidar pose

File: model/modelc_with_lidar.urdf (robot description, URDF)
Before this commit: robot whill_simulator, 12 links, 11 joints
Joints:
- joint left_lidar: origin xyz=0.535 0.215 0.35 rpy=0 0 1.5707 -> xyz=0.5 0.245 0.28 rpy=0 0 1.5707
- joint right_lidar: origin xyz=0.535 -0.215 0.35 rpy=0 0 -1.5707 -> xyz=0.5 -0.245 0.28 rpy=0 0 -1.5707

Commit message: Added mppi shared controller

File: model/modelc_with_lidar.urdf (robot description, URDF)
Before this commit: robot whill_simulator, 12 links, 11 joints
Joints:
- joint left_lidar: origin xyz=0.5 0.245 0.28 rpy=0 0 1.5707 -> xyz=0.5 0.255 0.28 rpy=0 0 1.5707
- joint right_lidar: origin xyz=0.5 -0.245 0.28 rpy=0 0 -1.5707 -> xyz=0.5 -0.255 0.28 rpy=0 0 -1.5707

Commit message: Added global planner into the controller support

File: model/modelc_with_lidar.urdf (robot description, URDF)
Before this commit: robot whill_simulator, 12 links, 11 joints
Joints:
- joint left_lidar: origin xyz=0.5 0.255 0.28 rpy=0 0 1.5707 -> xyz=0.5 0.28 0.28 rpy=0 0 1.5707
- joint right_lidar: origin xyz=0.5 -0.255 0.28 rpy=0 0 -1.5707 -> xyz=0.5 -0.28 0.28 rpy=0 0 -1.5707

Commit message: Working commit with Navfn path planner included to MPPI controller

File: model/modelc_with_lidar.urdf (robot description, URDF)
Before this commit: robot whill_simulator, 12 links, 11 joints
Joints:
- joint left_lidar: origin xyz=0.5 0.255 0.28 rpy=0 0 1.5707 -> xyz=0.5 0.250 0.28 rpy=0 0 1.5707
- joint right_lidar: origin xyz=0.5 -0.255 0.28 rpy=0 0 -1.5707 -> xyz=0.5 -0.250 0.28 rpy=0 0 -1.5707
